File: WRIP-ELECTRONICS/WRIP.kicad_pcb (KiCad board)
At the start: 2 copper layers, 7 x 35.8 mm, 25 parts, among them J1 Conn_01x02_Pin, J2 USB4145-03-0070-C_REVA2, J3 Conn_01x02_Pin, J4 Conn_01x01_Pin, J5 Conn_01x01_Pin, J6 Conn_01x01_Pin, J7 Conn_01x01_Pin, J8 Conn_01x01_Pin, SW1 SW_Push

Commit message: latest push
Parts:
- removed J2: USB4145-03-0070-C_REVA2, USB4145-03-0070-C_REVA2:GCT_USB4145-03-0070-C_REVA2
- removed R3, R4: 5.1k, Resistor_SMD:R_0402_1005Metric
- moved J1 16.2 mm to (69.2, 129.7), turned to 180 degrees
- moved C1 1.45 mm to (68.9, 118.2), turned to 180 degrees
Routing:
- net Net-(U1-VBUS): track 25.5 -> 1.98 mm, vias 2 -> 1
- net GND: track 35.0 -> 15.2 mm
- net Net-(J1-Pin_1): track 11.1 -> 8.33 mm
- net Net-(J2-CC2): track 2.46 -> 0.00 mm, vias 1 -> 0
- net Net-(J2-CC1): track 2.10 -> 0.00 mm, vias 1 -> 0
- net /vbat: track 36.4 -> 35.2 mm
- net Net-(D1-K): track 11.7 -> 10.6 mm
Other:
- board size 7 x 35.8 mm -> 7 x 25.5 mm
