File: WRIP-ELECTRONICS/WRIP.kicad_sch (KiCad schematic)
At the start: 19 parts, among them J1 Conn_01x02_Pin, J2 USB4145-03-0070-C_REVA2, SW1 SW_Push

Commit message: pcb
Parts:
- added J3: Conn_01x02_Pin, Connector_PinHeader_2.00mm:PinHeader_1x02_P2.00mm_Vertical, symbol Connector:Conn_01x02_Pin
- added J4, J5, J6, J7, J8: Conn_01x01_Pin, Connector_Pin:Pin_D1.0mm_L10.0mm_LooseFit, symbol Connector:Conn_01x01_Pin
- D1, D2, D3, D4: footprint (none) -> LED_SMD:LED_0402_1005Metric
- J1: footprint (none) -> Connector_PinHeader_2.00mm:PinHeader_1x02_P2.00mm_Vertical
- J2: footprint GCT_USB4145-03-0070-C_REVA2 -> USB4145-03-0070-C_REVA2:GCT_USB4145-03-0070-C_REVA2
- R1: footprint (lib_symbols -> Resistor_SMD:R_0402_1005Metric
- SW1: footprint (none) -> Button_Switch_SMD:SW_SPST_TL3342
- U1: footprint (none) -> Package_DFN_QFN:WQFN-24-1EP_4x4mm_P0.5mm_EP2.6x2.6mm_ThermalVias
Connections:
- net GND: now also J3.2 (Pin_2), J6.1 (Pin_1), J8.1 (Pin_1)
- net vbat: now also J3.1 (Pin_1), J4.1 (Pin_1)
- net 5v: now reaches C4.1, U1.17 (USBOUT1), U1.18 (USBOUT1)
- new net coil: J5.1 (Pin_1), J7.1 (Pin_1)

Commit message: ih
Parts:
- removed J2: USB4145-03-0070-C_REVA2, USB4145-03-0070-C_REVA2:GCT_USB4145-03-0070-C_REVA2, symbol USB4145-03-0070-C_REVA2:USB4145-03-0070-C_REVA2
- removed R3, R4: 5.1k, Resistor_SMD:R_0402_1005Metric, symbol Device:R
Connections:
- no-connect marks 11 -> 5
Changed lines of the file:
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@@
   (junction (at 179.07 82.55) (diameter 0) (color 0 0 0 0)
   )
-  (junction (at 212.09 29.21) (diameter 0) (color 0 0 0 0)
-  )
   (junction (at 170.18 82.55) (diameter 0) (color 0 0 0 0)
   )
@@
   (junction (at 170.18 72.39) (diameter 0) (color 0 0 0 0)
   )
-  (junction (at 172.72 29.21) (diameter 0) (color 0 0 0 0)
-  )
   (junction (at 156.21 72.39) (diameter 0) (color 0 0 0 0)
   )
@@
   (junction (at 170.18 64.77) (diameter 0) (color 0 0 0 0)
   )
-  (junction (at 212.09 62.23) (diameter 0) (color 0 0 0 0)
-  )
-  (junction (at 212.09 55.88) (diameter 0) (color 0 0 0 0)
-  )
   (junction (at 175.26 90.17) (diameter 0) (color 0 0 0 0)
   )
   (no_connect (at 130.81 85.09))
-  (no_connect (at 247.65 43.18))
-  (no_connect (at 212.09 45.72))
-  (no_connect (at 247.65 40.64))
   (no_connect (at 130.81 77.47))
   (no_connect (at 156.21 85.09))
-  (no_connect (at 247.65 45.72))
-  (no_connect (at 212.09 48.26))
   (no_connect (at 130.81 80.01))
   (no_connect (at 156.21 87.63))
-  (no_connect (at 212.09 43.18))
   (wire (pts (xy 104.14 53.34) (xy 104.14 62.23))
     (stroke (width 0) (type default))
   )
-  (wire (pts (xy 247.65 62.23) (xy 212.09 62.23))
-    (stroke (width 0) (type default))
-  )
   (wire (pts (xy 130.81 69.85) (xy 111.76 69.85))
     (stroke (width 0) (type default))
@@
     (stroke (width 0) (type default))
   )
-  (wire (pts (xy 256.54 50.8) (xy 256.54 48.26))
-    (stroke (width 0) (type default))
-  )
   (wire (pts (xy 104.14 62.23) (xy 130.81 62.23))
     (stroke (width 0) (type default))
@@
     (stroke (width 0) (type default))
   )
-  (wire (pts (xy 200.66 40.64) (xy 200.66 41.91))
-    (stroke (width 0) (type default))
-  )
   (wire (pts (xy 156.21 64.77) (xy 156.21 67.31))
     (stroke (width 0) (type default))
@@
     (stroke (width 0) (type default))
   )
-  (wire (pts (xy 247.65 38.1) (xy 247.65 27.94))
-    (stroke (width 0) (type default))
-  )
   (wire (pts (xy 156.21 90.17) (xy 157.48 90.17))
     (stroke (width 0) (type default))
   )
-  (wire (pts (xy 212.09 62.23) (xy 212.09 55.88))
-    (stroke (width 0) (type default))
-  )
   (wire (pts (xy 179.07 74.93) (xy 179.07 82.55))
     (stroke (width 0) (type default))
@@
     (stroke (width 0) (type default))
   )
-  (wire (pts (xy 201.93 40.64) (xy 200.66 40.64))
-    (stroke (width 0) (type default))
-  )
   (wire (pts (xy 123.19 82.55) (xy 130.81 82.55))
     (stroke (width 0) (type default))
@@
     (stroke (width 0) (type default))
   )
-  (wire (pts (xy 209.55 40.64) (xy 212.09 40.64))
-    (stroke (width 0) (type default))
-  )
   (wire (pts (xy 156.21 29.21) (xy 172.72 29.21))
     (stroke (width 0) (type default))
@@
     (stroke (width 0) (type default))
   )
-  (wire (pts (xy 212.09 50.8) (xy 212.09 55.88))
-    (stroke (width 0) (type default))
-  )
-  (wire (pts (xy 212.09 29.21) (xy 212.09 38.1))
-    (stroke (width 0) (type default))
-  )
   (wire (pts (xy 128.27 90.17) (xy 130.81 90.17))
     (stroke (width 0) (type default))
@@
     (stroke (width 0) (type default))
   )
-  (wire (pts (xy 212.09 27.94) (xy 212.09 29.21))
-    (stroke (width 0) (type default))
-  )
-  (wire (pts (xy 247.65 27.94) (xy 212.09 27.94))
-    (stroke (width 0) (type default))
-  )
   (wire (pts (xy 130.81 67.31) (xy 110.49 67.31))
     (stroke (width 0) (type default))
@@
   )
   (wire (pts (xy 156.21 69.85) (xy 156.21 72.39))
-    (stroke (width 0) (type default))
-  )
-  (wire (pts (xy 172.72 29.21) (xy 212.09 29.21))
-    (stroke (width 0) (type default))
-  )
-  (wire (pts (xy 247.65 48.26) (xy 248.92 48.26))
-    (stroke (width 0) (type default))
-  )
-  (wire (pts (xy 247.65 50.8) (xy 247.65 62.23))
     (stroke (width 0) (type default))
   )
@@
     )
   )
-  (symbol (lib_id "Device:R") (at 252.73 48.26 90) (unit 1)
-    (in_bom yes) (on_board yes) (dnp no) (fields_autoplaced)
-    (property "Reference" "R4" (at 252.73 43.18 90)
-      (effects (font (size 1.27 1.27)))
-    )
-    (property "Value" "5.1k" (at 252.73 45.72 90)
-      (effects (font (size 1.27 1.27)))
-    )
-    (property "Footprint" "Resistor_SMD:R_0402_1005Metric" (at 252.73 50.038 90)
-      (effects (font (size 1.27 1.27)) hide)
-    )
-    (property "Datasheet" "" (at 252.73 48.26 0)
-      (effects (font (size 1.27 1.27)) hide)
-    )
-    (pin "1")
-    (pin "2")
-    (instances
-      (project "WRIP"
-        (path "/82d3d878-b673-4943-8b42-48f483adab97"
-          (reference "R4") (unit 1)
-        )
-      )
-    )
-  )
   (symbol (lib_id "Connector:Conn_01x01_Pin") (at 95.25 123.19 180) (unit 1)
     (in_bom yes) (on_board yes) (dnp no) (fields_autoplaced)
@@
     )
   )
-  (symbol (lib_id "power:GND") (at 200.66 41.91 0) (unit 1)
-    (in_bom yes) (on_board yes) (dnp no) (fields_autoplaced)
-    (property "Reference" "#PWR010" (at 200.66 48.26 0)
-      (effects (font (size 1.27 1.27)) hide)
-    )
-    (property "Value" "GND" (at 200.66 46.99 0)
-      (effects (font (size 1.27 1.27)))
-    )
-    (property "Footprint" "" (at 200.66 41.91 0)
-      (effects (font (size 1.27 1.27)) hide)
-    )
-    (property "Datasheet" "" (at 200.66 41.91 0)
-      (effects (font (size 1.27 1.27)) hide)
-    )
-    (pin "1")
-    (instances
-      (project "WRIP"
-        (path "/82d3d878-b673-4943-8b42-48f483adab97"
-          (reference "#PWR010") (unit 1)
-        )
-      )
-    )
-  )
   (symbol (lib_id "Connector:Conn_01x02_Pin") (at 86.36 53.34 0) (unit 1)
     (in_bom yes) (on_board yes) (dnp no) (fields_autoplaced)
@@
         (path "/82d3d878-b673-4943-8b42-48f483adab97"
           (reference "J3") (unit 1)
-        )
-      )
-    )
-  )
-  (symbol (lib_id "USB4145-03-0070-C_REVA2:USB4145-03-0070-C_REVA2") (at 229.87 45.72 0) (unit 1)
-    (in_bom yes) (on_board yes) (dnp no) (fields_autoplaced)
-    (property "Reference" "J2" (at 229.87 31.75 0)
-      (effects (font (size 1.27 1.27)))
-    )
-    (property "Value" "USB4145-03-0070-C_REVA2" (at 229.87 34.29 0)
-      (effects (font (size 1.27 1.27)))
-    )
-    (property "Footprint" "USB4145-03-0070-C_REVA2:GCT_USB4145-03-0070-C_REVA2" (at 229.87 45.72 0)
-      (effects (font (size 1.27 1.27)) (justify bottom) hide)
-    )
-    (property "Datasheet" "" (at 229.87 45.72 0)
-      (effects (font (size 1.27 1.27)) hide)
-    )
-    (property "PARTREV" "A2" (at 229.87 45.72 0)
-      (effects (font (size 1.27 1.27)) (justify bottom) hide)
-    )
-    (property "STANDARD" "Manufacturer Recommendations" (at 229.87 45.72 0)
-      (effects (font (size 1.27 1.27)) (justify bottom) hide)
-    )
-    (property "SNAPEDA_PN" "USB4145-03-0070-C" (at 229.87 45.72 0)
-      (effects (font (size 1.27 1.27)) (justify bottom) hide)
-    )
-    (property "MAXIMUM_PACKAGE_HEIGHT" "7.66mm" (at 229.87 45.72 0)
-      (effects (font (size 1.27 1.27)) (justify bottom) hide)
-    )
-    (property "MANUFACTURER" "GCT" (at 229.87 45.72 0)
-      (effects (font (size 1.27 1.27)) (justify bottom) hide)
-    )
-    (pin "A1")
-    (pin "A12")
-    (pin "A4")
-    (pin "A5")
-    (pin "A6")
-    (pin "A7")
-    (pin "A8")
-    (pin "A9")
-    (pin "B1")
-    (pin "B12")
-    (pin "B4")
-    (pin "B5")
-    (pin "B6")
-    (pin "B7")
-    (pin "B8")
-    (pin "B9")
-    (pin "S1")
-    (pin "S2")
-    (pin "S3")
-    (pin "S4")
-    (instances
-      (project "WRIP"
-        (path "/82d3d878-b673-4943-8b42-48f483adab97"
-          (reference "J2") (unit 1)
         )
       )
@@
     )
   )
-  (symbol (lib_id "Device:R") (at 205.74 40.64 90) (unit 1)
-    (in_bom yes) (on_board yes) (dnp no) (fields_autoplaced)
-    (property "Reference" "R3" (at 205.74 35.56 90)
-      (effects (font (size 1.27 1.27)))
-    )
-    (property "Value" "5.1k" (at 205.74 38.1 90)
-      (effects (font (size 1.27 1.27)))
-    )
-    (property "Footprint" "Resistor_SMD:R_0402_1005Metric" (at 205.74 42.418 90)
-      (effects (font (size 1.27 1.27)) hide)
-    )
-    (property "Datasheet" "" (at 205.74 40.64 0)
-      (effects (font (size 1.27 1.27)) hide)
-    )
-    (pin "1")
-    (pin "2")
-    (instances
-      (project "WRIP"
-        (path "/82d3d878-b673-4943-8b42-48f483adab97"
-          (reference "R3") (unit 1)
-        )
-      )
-    )
-  )
-  (symbol (lib_id "power:GND") (at 256.54 50.8 0) (unit 1)
-    (in_bom yes) (on_board yes) (dnp no) (fields_autoplaced)
-    (property "Reference" "#PWR09" (at 256.54 57.15 0)
-      (effects (font (size 1.27 1.27)) hide)
-    )
-    (property "Value" "GND" (at 256.54 55.88 0)
-      (effects (font (size 1.27 1.27)))
-    )
-    (property "Footprint" "" (at 256.54 50.8 0)
-      (effects (font (size 1.27 1.27)) hide)
-    )
-    (property "Datasheet" "" (at 256.54 50.8 0)
-      (effects (font (size 1.27 1.27)) hide)
-    )
-    (pin "1")
-    (instances
-      (project "WRIP"
-        (path "/82d3d878-b673-4943-8b42-48f483adab97"
-          (reference "#PWR09") (unit 1)
-        )
-      )
-    )
-  )
   (symbol (lib_id "power:GND") (at 170.18 64.77 180) (unit 1)
     (in_bom yes) (on_board yes) (dnp no) (fields_autoplaced)
@@
         )
       )
-    )
-  )
-  (symbol (lib_id "power:GND") (at 212.09 62.23 0) (unit 1)
-    (in_bom yes) (on_board yes) (dnp no) (fields_autoplaced)
-    (property "Reference" "#PWR08" (at 212.09 68.58 0)
-      (effects (font (size 1.27 1.27)) hide)
-    )
-    (property "Value" "GND" (at 212.09 67.31 0)
-      (effects (font (size 1.27 1.27)))
-    )
-    (property "Footprint" "" (at 212.09 62.23 0)
-      (effects (font (size 1.27 1.27)) hide)
-    )
-    (property "Datasheet" "" (at 212.09 62.23 0)
-      (effects (font (size 1.27 1.27)) hide)
-    )
-    (pin "1")
-    (instances
-      (project "WRIP"
-        (path "/82d3d878-b673-4943-8b42-48f483adab97"
-          (reference "#PWR08") (unit 1)
-        )
-      )

Commit message: JBH
Parts:
- added R34: 30k, Resistor_SMD:R_0603_1608Metric, symbol Device:R
- added R37, R38: 1k, Resistor_SMD:R_0603_1608Metric, symbol Device:R
- added U5: TP4056, Package_SO:SOIC-8-1EP_3.9x4.9mm_P1.27mm_EP2.41x3.3mm_ThermalVias, symbol 1_sfxer symbols:IC_Battery_Management{colon}SOP-8_TP4056
Connections:
- net GND: now also R34.1, U5.1 (TEMP), U5.3 (GND), U5.9 (EP)
- new net: R34.2, U5.2 (PROG)
- new net: R37.1, U5.6 (~{STDBY})
- new net: R38.1, U5.7 (~{CHRG})
- new net +5V: U5.4 (VCC), U5.8 (CE)
- new net B+: U5.5 (BAT)
- new net CHG: R38.2
- new net FULL: R37.2
Other:
- note added: "BATTERY MANAGEMENT"
