File: WRIP-ELECTRONICS usb/WRIP-ELECTRONICS usb.kicad_pcb (KiCad board)
At the start: 2 copper layers, 5 parts

Commit message: h
Other:
- board outline added: 10.2 x 7 mm
Changed lines of the file:
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@@
       (net 8 "/vin"))
   )
-  (gr_rect (start 89.75 62) (end 100.25 69.5)
-    (stroke (width 0.1) (type default)) (fill none) (layer "F.Fab"))
+  (gr_rect (start 89.9 62) (end 100.12 68.98)
+    (stroke (width 0.1) (type default)) (fill none) (layer "Edge.Cuts"))
   (segment (start 94.250497 64.25) (end 93.75 63.749503) (width 0.25) (layer "F.Cu") (net 1))
   (segment (start 93.75 63.749503) (end 93.75 62.975) (width 0.25) (layer "F.Cu") (net 1))

Commit message: latest push
Other:
- board size 10.2 x 7 mm -> 9.7 x 6.5 mm
Changed lines of the file:
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@@
     (pad "B12" smd rect (at -3.2 -7.4) (size 0.6 1.2) (layers "F.Cu" "F.Paste" "F.Mask")
       (net 2 "GND") (pinfunction "GND") (pintype "passive") (thermal_bridge_angle 45))
-    (model "D:/sfxer/design/keyboard/components/3d models/hro_type-c-31-m-12.step"
+    (model "D:/sfxer/design/keyboard/components/3d models/hro_type-c-31-m-12.step" hide
       (offset (xyz -4.5 0 0))
       (scale (xyz 1 1 1))
@@
       (net 8 "/vin"))
   )
-  (gr_rect (start 89.9 62) (end 100.12 68.98)
+  (gr_rect (start 90.15 62.25) (end 99.87 68.73)
     (stroke (width 0.1) (type default)) (fill none) (layer "Edge.Cuts"))
   (segment (start 94.250497 64.25) (end 93.75 63.749503) (width 0.25) (layer "F.Cu") (net 1))
